Commit message: Update torso and change to Jax

File: assets/humanoid.urdf (robot description, URDF)
Before this commit: robot simple_humanoid, 15 links, 12 joints
Joints:
- added joint torso_to_right_hip_joint: type revolute, parent base_link, child right_upper_leg_link, origin xyz=0 0.1 -0.15 rpy=0 0 0, axis 1 0 0, limit lower=-1.57 upper=1.57 effort=15.0 velocity=1.0
- added joint torso_to_right_shoulder_joint: type revolute, parent upper_torso_link, child right_upper_arm_link, origin xyz=0 0.25 0.05 rpy=0 0 0, axis 1 0 0, limit lower=-1.57 upper=1.57 effort=10.0 velocity=1.0
